File: left.sch (KiCad schematic (older format))
At the start: 86 parts, among them J1 Buzzer, J11 Conn_01x01, J12 Conn_01x01, J13 Conn_01x01, J14 Conn_01x01, J15 Conn_01x01, J16 Conn_01x01, J17 Conn_01x01, J2 reset, J3 ISP, J7 Conn_01x01, J9 UTC16-G, P3 WS2812, P4 SJ-43514-SMT, SW1 Socket, SW10 Socket, SW11 Socket, SW12 Socket, SW13 Socket, SW14 Socket, SW15 Socket, SW16 Socket, SW17 Socket, SW18 Socket, SW19 Socket, SW2 Socket, SW20 Socket, SW21 Socket, SW22 Socket, SW23 Socket, SW24 Socket, SW3 Socket, SW4 Socket, SW49 FSMSM, SW5 Socket, SW6 Socket, SW7 Socket, SW8 Socket, SW9 Socket, U1 ATMega32U4, Y1 16MHz

Commit message: Added another row
Parts:
- added D13, D14, D15: BAV70, TO_SOT_Packages_SMD:SOT-23, symbol Device:D_x2_KCom_AAK
- added SW25, SW26, SW27, SW28, SW29, SW30: Socket, sockets:Kailh-socket, symbol Switch:SW_Push
- U1: symbol 8Bit-MCU:ATMega32U4 -> vitamins_included-rescue:ATMega32U4-8Bit-MCU
Connections:
- net labels added: row4
- wire segments 290 -> 308
Other:
- moved on the sheet: C10, C11, C12, C13, C14, C9, D1, D10, D11, D12, D2, D29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
