File: right.sch (KiCad schematic (older format))
At the start: 82 parts, among them J10 UTC16-G, J18 Conn_01x01, J19 Conn_01x01, J20 Conn_01x01, J21 Conn_01x01, J22 Conn_01x01, J23 Conn_01x01, J24 Conn_01x01, J4 reset, J5 Buzzer, J6 ISP, J8 Conn_01x01, P6 WS2812, P8 SJ-43514-SMT, SW25 Socket, SW26 Socket, SW27 Socket, SW28 Socket, SW29 Socket, SW30 Socket, SW31 Socket, SW32 Socket, SW33 Socket, SW34 Socket, SW35 Socket, SW36 Socket, SW37 Socket, SW38 Socket, SW39 Socket, SW40 Socket, SW41 Socket, SW42 Socket, SW43 Socket, SW44 Socket, SW45 Socket, SW46 Socket, SW47 Socket, SW48 Socket, SW50 FSMSM, U2 ATMega32U4, Y2 16MHz

Commit message: Added another row
Parts:
- added D28, D29, D30: BAV70, TO_SOT_Packages_SMD:SOT-23, symbol Device:D_x2_KCom_AAK
- added SW55, SW56, SW57, SW58, SW59, SW60: Socket, sockets:Kailh-socket, symbol Switch:SW_Push
- U2: symbol 8Bit-MCU:ATMega32U4 -> vitamins_included-rescue:ATMega32U4-8Bit-MCU
- renumbered D13 to D16, D14 to D17, D15 to D18, D16 to D19, D17 to D20, D18 to D21, D19 to D22, D20 to D23, D21 to D24, D22 to D25, D23 to D26, D24 to D27, SW25 to SW31, SW26 to SW32, SW27 to SW33, SW28 to SW34, SW29 to SW35, SW30 to SW36, SW31 to SW37, SW32 to SW38, SW33 to SW39, SW34 to SW40, SW35 to SW41, SW36 to SW42, SW37 to SW43, SW38 to SW44, SW39 to SW45, SW40 to SW46, SW41 to SW47, SW42 to SW48, SW43 to SW49, SW44 to SW50, SW45 to SW51, SW46 to SW52, SW47 to SW53, SW48 to SW54
Connections:
- net labels added: row4
- wire segments 279 -> 297
Other:
- moved on the sheet: D16, D17, D18, D19, D20, D21, D22, D23, D24, D25, D26, D27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
